Commit message: gripper joint removed

File: urdf/robotiq_hande.urdf (robot description, URDF)
Before this commit: robot robotiq_hande, 4 links, 4 joints
Joints:
- joint hande_joint_finger: limit lower=0 upper=0.025 effort=130 velocity=0.15 -> (none); type prismatic -> fixed
- joint robotiq_hande_base_to_hande_right_finger: limit lower=0 upper=0.025 effort=130 velocity=0.15 -> (none); mimic joint=hande_joint_finger multiplier=1 offset=0 -> (none); type prismatic -> fixed
