Commit message: new shelf

File: urdf/shelf.urdf (robot description, URDF)
Before this commit: robot shelf, 7 links, 7 joints
Links:
- link stand_link: geometry collision box size=1.08 1.08 0.9; visual box size=1.08 1.08 0.9
Joints:
- joint shelf_joint: origin xyz=0 -0.5 0 rpy=0 0 3.14 -> xyz=0 -0.54 0 rpy=1.57 0 3.14

Commit message: auto cooking station collision turned off

File: urdf/shelf.urdf (robot description, URDF)
Before this commit: robot shelf, 7 links, 7 joints
Links:
- link station_link: geometry visual box size=0.4 0.4 0.26
